File: vco/vco.kicad_sch (KiCad schematic)
At the start: 0 parts

Commit message: Add vco
Parts:
- added C1: 2.2nF, symbol Device:C
- added C2, C3: 1uF, symbol Device:C
- added D1, D2, D3: 1N4148, Diode_THT:D_DO-35_SOD27_P7.62mm_Horizontal, symbol Diode:1N4148
- added J1: CV in, symbol Connector:Barrel_Jack
- added J2: FM in, symbol Connector:Barrel_Jack
- added J3: Saw_Out, symbol Connector:Barrel_Jack
- added J4: PWM_In, symbol Connector:Barrel_Jack
- added J5: Sq_Out, symbol Connector:Barrel_Jack
- added J6: Tri_Out, symbol Connector:Barrel_Jack
- added Q1: BC558, Package_TO_SOT_THT:TO-92_Inline, symbol Transistor_BJT:BC558
- added Q2: BC548, Package_TO_SOT_THT:TO-92_Inline, symbol Transistor_BJT:BC548
- added R1, R13, R3, R4, R7, R9: 100K, symbol Device:R_US
- added R10, R15, R16: 1K, symbol Device:R_US
- added R11: 14K, symbol Device:R_US
- added R12, R14: 68K, symbol Device:R_US
- added R17, R18: 10K, symbol Device:R_US
- added R19: 20K, symbol Device:R_US
- added R2, R6: 1M, symbol Device:R_US
- added R20: 200K, symbol Device:R_US
- added R5: 1K5, symbol Device:R_US
- added R8: 33K, symbol Device:R_US
- added RV1: 1K, symbol Device:R_Potentiometer_Trim_US
- added RV2: 250K, symbol Device:R_Potentiometer_Trim_US
- added RV_Coarse, RV_Duty, RV_Fine: 100K, symbol Device:R_Potentiometer_US
- added RV_FM: 1M, symbol Device:R_Potentiometer_US
- added TH1, TH2, TH3, TH4: 10K, symbol Device:Thermistor_NTC
- added U1: 40106, symbol 4xxx:40106
- added U2, U3: TL074, symbol Amplifier_Operational:TL074
Connections:
- new net: R11.1, R12.1, RV_Duty.2, U2.9 (-)
- new net: C3.1, D2.1 (K), D3.1 (K), R19.1
- new net: D2.2 (A), R17.1, U3.1, U3.2 (-)
- new net: C1.1, D1.1 (K), Q2.1 (C), U1.1
- new net: D1.2 (A), U1.2, U2.3 (+)
- new net: R5.2, RV1.1
- new net: J2.1, R4.1
- new net: R4.2, TH4.1
- new net: C2.2, R7.1, U2.10 (+), U2.5 (+), U3.3 (+)
- new net: R8.1, R9.1, U2.6 (-)
- new net: R10.1, R9.2, U2.7
- new net: J1.1, R3.1
- new net: R3.2, TH3.1
- new net: C3.2, R20.1, U3.10 (+)
- new net: R16.1, U3.8, U3.9 (-)
- new net: C2.1, U2.1, U2.2 (-)
- new net: Q1.2 (B), R5.1, RV_FM.2, RV_FM.3, TH1.2, TH2.2, TH3.2
- new net: J6.1, R16.2
- new net: J4.1, RV2.1
- new net: R12.2, RV2.2, RV2.3
- new net: R13.2, R14.1, U2.12 (+)
- new net: R15.1, U2.13 (-), U2.14
- new net: R2.1, RV_Fine.2
- new net: R2.2, TH2.1
- new net: J5.1, R15.2
- new net: R13.1, U2.8
- new net: R1.1, RV_Coarse.2
- new net: J3.1, R10.2
- new net: R1.2, TH1.1
- new net: D3.2 (A), R18.2, U3.7
- new net: RV_FM.1, TH4.2
- new net: Q1.1 (C), Q2.2 (B), R6.2
- new net: R17.2, R18.1, U3.6 (-)
- new net +12V: R6.1, RV_Duty.1
- new net -12V: Q1.3 (E), R19.2, RV_Coarse.3, RV_Duty.3, RV_Fine.3
- new net GND: C1.2, J1.2, J2.2, J3.2, J4.2, J5.2, J6.2, Q2.3 (E), R11.2, R14.2, R20.2, R7.2, R8.2, RV1.2, RV1.3, RV_Coarse.1, RV_Fine.1, U3.5 (+)
