File: adsr/adsr.kicad_sch (KiCad schematic)
At the start: 0 parts

Commit message: adr
Parts:
- added C1: 1uF, symbol Device:C
- added D1, D2, D3: 1N4148, Diode_THT:D_DO-35_SOD27_P7.62mm_Horizontal, symbol Diode:1N4148
- added J1, J2: Barrel_Jack, symbol Connector:Barrel_Jack
- added R1, R3: 100k, symbol Device:R_US
- added R2: 47k, symbol Device:R_US
- added R4: 1k, symbol Device:R_US
- added RV1, RV2: 1M, symbol Device:R_Potentiometer_US
- added U1: TL074, symbol Amplifier_Operational:TL074
Connections:
- new net: R1.2, R2.2, U1.2 (-)
- new net: D2.1 (K), D3.2 (A), U1.6 (-), U1.7
- new net: D2.2 (A), RV2.1
- new net: J2.1, R4.2
- new net: D3.1 (K), RV1.1
- new net: C1.1, RV1.2, RV1.3, RV2.2, RV2.3, U1.10 (+)
- new net: J1.1, U1.3 (+)
- new net: R4.1, U1.8, U1.9 (-)
- new net: D1.1 (K), R3.1, U1.5 (+)
- new net: D1.2 (A), U1.1
- new net +12V: R1.1
- new net GND: C1.2, J1.2, J2.2, R2.1, R3.2

Commit message: noise
Parts:
- added C2: 1uF, symbol Device:C
- added D4, D5: 1N4148, Diode_THT:D_DO-35_SOD27_P7.62mm_Horizontal, symbol Diode:1N4148
- added R5: 100k, symbol Device:R_US
- added R6: 10k, symbol Device:R_US
- added RV3: 100k, symbol Device:R_Potentiometer_US
- added U2: TL074, symbol Amplifier_Operational:TL074
Connections:
- net GND: now also R5.2, R6.2, RV3.3; no longer R3.2
- net at R1.2, R2.2, U1.2 (-): now also U2.2 (-)
- net at J1.1, U1.3 (+): now also C2.1
- net at R3.1, U1.5 (+): now also D4.1 (K); no longer D1.1 (K)
- new net: D1.1 (K), RV3.1
- new net: R3.2, RV3.2
- new net: D4.2 (A), U2.1
- new net: D5.1 (K), R5.1, U2.3 (+)
- new net: C2.2, D5.2 (A), R6.1
Other:
- moved on the sheet: C1, D1, D2, D3, J1, J2, R1, R2, R4, RV1, RV2, U1A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
